File: PCB/PCB.kicad_pcb (KiCad board)
At the start: 2 copper layers, 70 x 55 mm, 45 parts, among them J1 Conn_01x04_Pin, J2 Conn_01x01, J3 Conn_01x08, J4 Conn_01x02, J6 Conn_01x04, SW1 PTS815SJM250SMTRLFS, SW2 PTS815SJM250SMTRLFS, U1 IQS7222A001QNR, U6 AP63203WU, U7 ESP32-C3-WROOM-02

Commit message: commit
Parts:
- added U2: IRM-20-24, easyeda2kicad:PWRM-TH_IRM-20-24, F.Cu at (60.0, 117.5)
- J4: value Conn_01x02 -> 703W-00_53; footprint Connector_JST:JST_XH_B2B-XH-AM_1x02_P2.50mm_Vertical -> Extra:QUALTEK_703W-00_53
- moved J4 47.5 mm to (65.0, 97.5)
Connections:
- J4 pad 1: +24V -> N
- J4 pad 2: GND -> unconnected-(J4-EARTH-Pad2)
Routing:
- net L: track 0.00 -> 59.7 mm
- net +24V: track 33.4 -> 92.8 mm
- net N: track 0.00 -> 36.8 mm
Other:
- board size 70 x 55 mm -> 70 x 104.5 mm
